File: resividor 3.kicad_pcb (KiCad board)
At the start: 2 copper layers, 50.8 x 50.8 mm, 14 parts, among them J1 RJ45, J2 RJ45, J3 Screw_Terminal_01x02, J4 Screw_Terminal_01x02, J5 Screw_Terminal_01x02, Q1 IRLZ44N, Q2 IRLZ44N, Q3 IRLZ44N

Commit message: Add files via upload
Routing:
- net Net-(J1-Pad5): vias 0 -> 1
- net Net-(J1-Pad3): vias 0 -> 1
Changed lines of the file:
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@@
   (segment (start 81.28 74.1525) (end 81.28 78.74) (width 0.6) (layer "F.Cu") (net 9))
   (segment (start 81.28 78.74) (end 83.82 81.28) (width 0.6) (layer "F.Cu") (net 9))
+  (segment (start 83.913468 85.880248) (end 74.543716 95.25) (width 0.6) (layer "F.Cu") (net 9))
+  (segment (start 74.543716 95.25) (end 73.64 95.25) (width 0.6) (layer "F.Cu") (net 9))
   (segment (start 83.913468 81.28) (end 83.913468 85.880248) (width 0.6) (layer "F.Cu") (net 9))
   (segment (start 71.1 93.98) (end 72.37 93.98) (width 0.6) (layer "F.Cu") (net 9))
@@
   (segment (start 72.37 65.2425) (end 73.64 66.5125) (width 0.6) (layer "F.Cu") (net 9))
   (segment (start 72.37 93.98) (end 73.64 95.25) (width 0.6) (layer "F.Cu") (net 9))
-  (segment (start 83.82 85.973716) (end 83.913468 85.880248) (width 0.6) (layer "B.Cu") (net 9))
-  (segment (start 74.93 95.25) (end 83.82 86.36) (width 0.6) (layer "B.Cu") (net 9))
-  (segment (start 83.82 86.36) (end 83.82 85.973716) (width 0.6) (layer "B.Cu") (net 9))
-  (segment (start 73.64 95.25) (end 74.93 95.25) (width 0.6) (layer "B.Cu") (net 9))
   (segment (start 72.37 62.7025) (end 73.64 63.9725) (width 0.6) (layer "F.Cu") (net 10))
   (segment (start 83.913468 69.655809) (end 83.913468 71.12) (width 0.6) (layer "F.Cu") (net 10))
@@
   (segment (start 71.1 62.7025) (end 72.37 62.7025) (width 0.6) (layer "F.Cu") (net 10))
   (segment (start 72.37 91.44) (end 73.64 92.71) (width 0.6) (layer "F.Cu") (net 10))
-  (segment (start 74.93 92.71) (end 81.28 86.36) (width 0.6) (layer "B.Cu") (net 10))
+  (segment (start 74.93 92.71) (end 73.64 92.71) (width 0.6) (layer "F.Cu") (net 10))
+  (segment (start 81.28 86.36) (end 74.93 92.71) (width 0.6) (layer "F.Cu") (net 10))
+  (via (at 81.28 86.36) (size 0.8) (drill 0.4) (layers "F.Cu" "B.Cu") (net 10))
   (segment (start 81.28 77.298666) (end 83.913468 74.665198) (width 0.6) (layer "B.Cu") (net 10))
   (segment (start 81.28 86.36) (end 81.28 77.298666) (width 0.6) (layer "B.Cu") (net 10))
-  (segment (start 73.64 92.71) (end 74.93 92.71) (width 0.6) (layer "B.Cu") (net 10))
+  (segment (start 74.93 90.17) (end 73.64 90.17) (width 0.6) (layer "F.Cu") (net 11))
   (segment (start 73.64 61.4325) (end 83.3475 61.4325) (width 0.6) (layer "F.Cu") (net 11))
   (segment (start 83.82 58.42) (end 83.82 60.96) (width 0.6) (layer "F.Cu") (net 11))
   (segment (start 71.1 88.9) (end 72.37 88.9) (width 0.6) (layer "F.Cu") (net 11))
   (segment (start 72.37 88.9) (end 73.64 90.17) (width 0.6) (layer "F.Cu") (net 11))
+  (segment (start 78.74 86.36) (end 74.93 90.17) (width 0.6) (layer "F.Cu") (net 11))
   (segment (start 83.82 60.96) (end 83.82 63.5) (width 0.6) (layer "F.Cu") (net 11))
   (segment (start 71.1 60.1625) (end 72.37 60.1625) (width 0.6) (layer "F.Cu") (net 11))
   (segment (start 72.37 60.1625) (end 73.64 61.4325) (width 0.6) (layer "F.Cu") (net 11))
   (segment (start 83.3475 61.4325) (end 83.82 60.96) (width 0.6) (layer "F.Cu") (net 11))
-  (segment (start 74.93 90.17) (end 78.74 86.36) (width 0.6) (layer "B.Cu") (net 11))
+  (via (at 78.74 86.36) (size 0.8) (drill 0.4) (layers "F.Cu" "B.Cu") (net 11))
   (segment (start 78.74 76.2) (end 81.28 73.66) (width 0.6) (layer "B.Cu") (net 11))
   (segment (start 81.28 66.04) (end 83.82 63.5) (width 0.6) (layer "B.Cu") (net 11))
   (segment (start 78.74 86.36) (end 78.74 76.2) (width 0.6) (layer "B.Cu") (net 11))
   (segment (start 81.28 73.66) (end 81.28 66.04) (width 0.6) (layer "B.Cu") (net 11))
-  (segment (start 73.64 90.17) (end 74.93 90.17) (width 0.6) (layer "B.Cu") (net 11))
 )
