File: kicad/sender/sender.kicad_pcb (KiCad board)
At the start: 2 copper layers, 55.9 x 71.1 mm, 18 parts, among them J1 RJ45, J2 Screw_Terminal_01x03, J3 Conn_01x10_Pin, J4 Conn_01x08_Pin, J5 Conn_01x06_Pin, J6 Conn_01x08_Pin, Q1 IRLZ44N, Q2 IRLZ44N, Q3 IRLZ44N, U1 MAX481E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

Commit message: Add files via upload
Parts:
- removed J1: RJ45, Connector_RJ:RJ45_Amphenol_54602-x08_Horizontal
- added J7: Conn_01x04, Connector_PinHeader_2.54mm:PinHeader_1x04_P2.54mm_Vertical, F.Cu at (142.6, 94.9)
- added J8: Conn_01x04, Connector_PinHeader_2.54mm:PinHeader_1x04_P2.54mm_Vertical, F.Cu at (145.5, 96.5)
- moved J2 36.3 mm to (106.8, 93.4), turned to -90 degrees
Routing:
- net Net-(J2-Pin_3): track 65.8 -> 135.7 mm
- net Net-(J2-Pin_2): track 62.6 -> 112.4 mm, vias 0 -> 2
- net Net-(J2-Pin_1): track 188.1 -> 163.6 mm
- net Net-(J7-Pin_3): track 37.8 -> 49.2 mm, vias 0 -> 1
- net Net-(J7-Pin_2): track 34.3 -> 42.3 mm, vias 0 -> 1
- net Net-(J7-Pin_4): track 49.4 -> 57.3 mm, vias 0 -> 1
- net Net-(U2-C): track 13.0 -> 14.7 mm, vias 0 -> 1
- net Net-(J4-Pin_4): track 92.3 -> 91.1 mm, vias 0 -> 1
- net Net-(J6-Pin_3): track 11.0 -> 11.9 mm
- net Net-(U2-VO): track 18.1 -> 18.3 mm, vias 0 -> 1
Other:
- board size 55.9 x 71.1 mm -> 58.4 x 73.7 mm
